Commit message: Imported upstream version '0.1.2' of 'upstream'

File: grizzly_description/urdf/wheel.urdf.xacro (robot description, xacro)
@@ -106,7 +106,4 @@
           <cylinder length="${wheel_z_size}"
                     radius="${wheel_x_size/2}" />
-          <!--
-                    <mesh filename="package://husky_description/Media/models/wheel.stl" />
-                -->
         </geometry>
       </collision>
