Commit message: Imported upstream version '0.3.0' of 'upstream'

File: grizzly_description/urdf/base.urdf.xacro (robot description, xacro)
@@ -2,4 +2,5 @@
 <!--
 Copyright (c) 2012, Siddhant Ahuja (Sid), Ryan Gariepy
+Copyright (c) 2014, Clearpath Robotics
 All rights reserved.
 Redistribution and use in source and binary forms, with or without
@@ -25,187 +26,121 @@
 This program contains the description of the robot base model for the Clearpath Grizzly
 -->
-<robot xmlns:xi="http://www.w3.org/2001/XInclude"
-       xmlns:gazebo="http://playerstage.sourceforge.net/gazebo/xmlschema/#gz"
-       xmlns:model="http://playerstage.sourceforge.net/gazebo/xmlschema/#model"
-       xmlns:sensor="http://playerstage.sourceforge.net/gazebo/xmlschema/#sensor"
-       xmlns:body="http://playerstage.sourceforge.net/gazebo/xmlschema/#body"
-       xmlns:geom="http://playerstage.sourceforge.net/gazebo/xmlschema/#geom"
-       xmlns:joint="http://playerstage.sourceforge.net/gazebo/xmlschema/#joint"
-       xmlns:controller="http://playerstage.sourceforge.net/gazebo/xmlschema/#controller"
-       xmlns:interface="http://playerstage.sourceforge.net/gazebo/xmlschema/#interface"
-       xmlns:rendering="http://playerstage.sourceforge.net/gazebo/xmlschema/#rendering"
-       xmlns:renderable="http://playerstage.sourceforge.net/gazebo/xmlschema/#renderable"
-       xmlns:physics="http://playerstage.sourceforge.net/gazebo/xmlschema/#physics"
-       xmlns:xacro="http://ros.org/wiki/xacro"
-       name="grizzly">
+<robot name="grizzly" xmlns:xacro="http://www.ros.org/wiki/xacro">
+  <property name="M_PI" value="3.1415926535897931" />
+  <property name="ground_clearance" value="0.203" />
   <!-- Included URDF/XACRO Files -->
-  <xacro:include filename="$(find grizzly_description)/urdf/materials.urdf.xacro" />
-  <xacro:include filename="$(find grizzly_description)/urdf/wheel.urdf.xacro" />
-  <xacro:include filename="$(find grizzly_description)/urdf/parts.urdf.xacro" />
-  <xacro:include filename="$(find grizzly_description)/urdf/add_frame.urdf.xacro" />
-  <!-- PROPERTY LIST -->
-  <!--All units in m-kg-s-radians unit system -->
-  <property name="M_PI"
-            value="3.1415926535897931" />
-  <!-- Main Body-base-->
-  <!-- Location of com : center of mass -->
-  <property name="base_x_com"
-            value="-0.08748000" />
-  <property name="base_y_com"
-            value="-0.00085000" />
-  <property name="base_z_com"
-            value="0.09947000" />
-  <!-- Size of the base-->
-  <property name="base_x_size"
-            value="0.708" />
-  <property name="base_y_size"
-            value="0.3" />
-  <property name="base_z_size"
-            value="1.826" />
-  <!--Weight of the base-->
-  <property name="base_mass"
-            value="33.45489000" />
-  <!-- in kg-->
-  <!--Weight of the front axle-->
-  <property name="front_axle_mass"
-            value="0.45489000" />
-  <!-- in kg-->
-  <!--Inertial values for the front_axle at center of mass, aligned with coordinate system. Units are kg*m^2-->
-  <property name="front_axle_ixx_com_cs"
-            value="0.60216370" />
-  <property name="front_axle_ixy_com_cs"
-            value="-0.02364198" />
-  <property name="front_axle_ixz_com_cs"
-            value="-0.11972132" />
-  <property name="front_axle_iyy_com_cs"
-            value="1.73859574" />
-  <property name="front_axle_iyz_com_cs"
-            value="-0.00154437" />
-  <property name="front_axle_izz_com_cs"
-            value="2.02955229" />
-  <!--Inertial values for the base at center of mass, aligned with coordinate system. Units are kg*m^2-->
-  <property name="base_ixx_com_cs"
-            value="0.60216370" />
-  <property name="base_ixy_com_cs"
-            value="-0.02364198" />
-  <property name="base_ixz_com_cs"
-            value="-0.11972132" />
-  <property name="base_iyy_com_cs"
-            value="1.73859574" />
-  <property name="base_iyz_com_cs"
-            value="-0.00154437" />
-  <property name="base_izz_com_cs"
-            value="2.02955229" />
-  <!-- BASE-FOOTPRINT -->
-  <!-- base_footprint is a fictitious link(frame) that is on the ground right below base_link origin, navigation stack depends on this frame -->
-  <link name="base_footprint">
+  <xacro:include filename="materials.urdf.xacro" />
+  <xacro:include filename="wheel.urdf.xacro" />
+  <xacro:include filename="grizzly.gazebo" />
+  <!-- Key Dimensions -->
+  <property name="chassis_length" value="1.75" />
+  <property name="chassis_width" value="0.711" />
+  <property name="chassis_height" value="0.495" />
+  <property name="chassis_mass" value="487" />
+  <property name="front_axle_mass" value="113" />
+  <property name="front_axle_radius" value="0.13" />
+  <property name="front_axle_length" value="1.0" />
+  <property name="base_x_origin_to_wheel_origin" value="0.448" /> <!-- 240/2 + 660/2-->
+  <property name="base_y_origin_to_wheel_origin" value="0.499" /> <!--(1282-711)/4 + 711/2-->
+  <property name="base_z_origin_to_wheel_origin" value="0.0" />
+  <!-- Root link of Grizzly -->
+  <link name="base_link" />
+  <!-- Actual body/chassis of the robot, separate from base_link due to KDL inertia issue. -->
+  <link name="chassis_link">
     <inertial>
-      <mass value="0.0001" />
-      <origin xyz="0 0 0" />
-      <inertia ixx="0.0001"
-               ixy="0.0"
-               ixz="0.0"
-               iyy="0.0001"
-               iyz="0.0"
-               izz="0.0001" />
+      <mass value="${chassis_mass}"/>
+      <origin xyz="-0.013 -0.00061 -0.0205"/>
+      <inertia ixx="64.010712692" ixy="0.214224647" ixz="-1.636784296"
+               iyy="200.87" iyz="-0.048325439" izz="229.831441333" />
     </inertial>
     <visual>
-      <origin xyz="0 0 0"
-              rpy="0 0 0" />
-      <geometry>
-        <box size="0.001 0.001 0.001" />
-      </geometry>
-    </visual>
-  </link>
-  <gazebo reference="base_footprint">
-    <turnGravityOff>false</turnGravityOff>
-  </gazebo>
-  <joint name="base_footprint_joint"
-         type="fixed">
-    <origin xyz="0 0 ${wheel_x_size/2}"
-            rpy="0 0 0" />
-    <parent link="base_footprint" />
-    <child link="base_link" />
-  </joint>
-  <!-- BASE-LINK -->
-  <!--Actual body/chassis of the robot-->
-  <link name="base_link">
-    <inertial>
-      <mass value="${base_mass}" />
-      <!--This is the pose of the inertial reference frame, relative to the link reference frame. The origin of the inertial reference frame needs to be at the center of gravity. The axes of the inertial reference frame do not need to be aligned with the principal axes of the inertia.-->
-      <origin xyz="${base_x_com} ${base_y_com} ${base_z_com}" />
-      <!--The 3x3 rotational inertia matrix. Because the rotational inertia matrix is symmetric, only 6 above-diagonal elements of this matrix are specified here, using the attributes ixx, ixy, ixz, iyy, iyz, izz.-->
-      <inertia ixx="${base_ixx_com_cs}"
-               ixy="${base_ixy_com_cs}"
-               ixz="${base_ixz_com_cs}"
-               iyy="${base_iyy_com_cs}"
-               iyz="${base_iyz_com_cs}"
-               izz="${base_izz_com_cs}" />
-    </inertial>
-    <visual>
-      <origin xyz="0 0 ${base_z_origin_offset}"
+      <origin xyz="0 0 ${ground_clearance}"
               rpy="${M_PI/2} 0 ${M_PI/2}" />
       <geometry>
         <mesh filename="package://grizzly_description/meshes/base_link.stl" />
       </geometry>
-      <material name="Black" />
+      <material name="DarkGrey" />
     </visual>
     <collision>
-      <origin xyz="0 0 0.3"
+      <origin xyz="0 0 ${ground_clearance}"
               rpy="${M_PI/2} 0 ${M_PI/2}" />
       <geometry>
-        <box size="${base_x_size} ${base_y_size} ${base_z_size}" />
-        <!--making it slightly bigger in x and z direction-->
+         <box size="${chassis_width} ${chassis_height} ${chassis_length}" />
       </geometry>
     </collision>
   </link>
-  <gazebo reference="base_link">
-    <material>Gazebo/FlatBlack</material>
-    <turnGravityOff>false</turnGravityOff>
-  </gazebo>
+  <joint name="chassis_joint"
+         type="fixed">
+    <origin xyz="0 0 ${ground_clearance}"
+            rpy="0 0 0"/>
+    <parent link="base_link" />
+    <child link="chassis_link" />
+  </joint>
   <!-- Add a sensor anchor link that points to the center of the robot top plate -->
-  <grizzly_tf parent="base_link" name="sensor_anchor_link"
-    translateX="0" translateY="0" translateZ="0.45"
-    rotateX="0.0" rotateY="0.0" rotateZ="0.0"/>
-  <!-- Add a sensor anchor link for the imu -->
-  <grizzly_tf parent="sensor_anchor_link" name="imu_link"
-    translateX="-0.788" translateY="0" translateZ="-0.118"
-    rotateX="3.1415" rotateY="1.5701" rotateZ="0" />
-  <!-- DECORATIONS -->
-  <!-- Bumpers -->
-  <grizzly_part parent="base_footprint"
-                name="bumper"
-                mesh="bumper"
-                colour="Yellow"
-                translateX="0.0"
-                translateY="0.0"
-                translateZ="0.5"
-                rotateX="${M_PI/2}"
-                rotateY="0.0"
-                rotateZ="${M_PI/2}" />
-  <gazebo reference="base_footprint_bumper_part">
-    <material>Gazebo/Yellow</material>
-  </gazebo>
-  <!-- Back wheels -->
-  <grizzly_wheel fb="back"
-                 lr="left"
-                 parent="base_link"
-                 translateX="-1.75"
-                 translateY="1.75"
-                 translateZ="0"
-                 flipY="0" />
-  <grizzly_wheel fb="back"
-                 lr="right"
-                 parent="base_link"
-                 translateX="-1.75"
-                 translateY="-1.75"
-                 translateZ="0"
-                 flipY="1" />
-  <!-- Front axle link -->
+  <link name="sensor_anchor_link"/>
+  <joint name="sensor_anchor_joint" type="fixed">
+    <origin xyz="0 0 ${chassis_height}"
+            rpy="0 0 0" />
+    <parent link="chassis_link" />
+    <child link="sensor_anchor_link" />
+  </joint>
+  <!-- This is the approximate position of the GPS antenna on the standard configuration. -->
+  <link name="navsat_link" />
+  <joint name="navsat_joint" type="fixed">
+    <origin xyz="-${chassis_length/2} 0 0"
+            rpy="0 0 0" />
+    <parent link="sensor_anchor_link" />
+    <child link="navsat_link" />
+  </joint>
+  <!-- The position and orientation of the IMU in the rear compartment. -->
+  <link name="imu_link" />
+  <joint name="imu_joint" type="fixed">
+    <origin xyz="-${chassis_length/2} 0 -${chassis_height/2}"
+             rpy="${M_PI} ${M_PI/2} 0" />
+    <parent link="sensor_anchor_link" />
+    <child link="imu_link" />
+  </joint>
+  <!-- Purely decorative visual component. -->
+  <link name="fenders_link">
+    <visual>
+      <origin xyz="0 0 ${ground_clearance}" rpy="${M_PI/2} 0 ${M_PI/2}"/>
+      <geometry>
+        <mesh filename="package://grizzly_description/meshes/bumper.stl" />
+      </geometry>
+      <material name="Yellow" />
+    </visual>
+  </link>
+  <joint name="fenders_joint" type="fixed">
+    <parent link="chassis_link" />
+    <child link="fenders_link" />
+  </joint>
+  <link name="front_axle_link">
+    <inertial>
+      <mass value="${front_axle_mass}" />
+      <origin xyz="0 0 0"/>
+      <inertia ixx="9.9" ixy="0.0" ixz="0.0" iyy="9.9" iyz="0.0" izz="0.95" />
+    </inertial>
+    <visual>
+      <origin xyz="-${ground_clearance} 0 ${base_y_origin_to_wheel_origin}"
+              rpy="0 ${M_PI} ${M_PI/2}" />
+      <geometry>
+        <mesh filename="package://grizzly_description/meshes/front_axle.stl" />
+      </geometry>
+      <material name="DarkGrey" />
+    </visual>
+    <collision>
+      <origin xyz="0 0 0"
+              rpy="${M_PI/2} 0 0" />
+      <geometry>
+        <cylinder length="${front_axle_length}"
+                  radius="${front_axle_radius}" />
+      </geometry>
+    </collision>
+  </link>
   <joint name="front_axle_joint"
          type="revolute">
-    <origin xyz="0.4375 0 0"
+    <origin xyz="${base_x_origin_to_wheel_origin} 0 0"
             rpy="0 0 0" />
-    <parent link="base_link" />
+    <parent link="chassis_link" />
     <child link="front_axle_link" />
     <axis xyz="1 0 0"
@@ -216,66 +151,11 @@
            velocity="0.5" />
   </joint>
-  <link name="front_axle_link">
-    <inertial>
-      <mass value="${front_axle_mass}" />
-      <origin xyz="0 0 0" />
-      <inertia ixx="${front_axle_ixx_com_cs}"
-               ixy="${front_axle_ixy_com_cs}"
-               ixz="${front_axle_ixz_com_cs}"
-               iyy="${front_axle_iyy_com_cs}"
-               iyz="${front_axle_iyz_com_cs}"
-               izz="${front_axle_izz_com_cs}" />
-    </inertial>
-    <visual>
-      <origin xyz="-0.2 0 0.45"
-              rpy="0 ${M_PI} ${M_PI/2}" />
-      <geometry>
-        <mesh filename="package://grizzly_description/meshes/front_axle.stl" />
-      </geometry>
-      <material name="Black" />
-    </visual>
-    <collision>
-      <origin xyz="0 0 0"
-              rpy="${M_PI/2} 0 0" />
-      <geometry>
-        <cylinder length="1.0"
-                  radius="0.13" />
-      </geometry>
-    </collision>
-  </link>
-  <gazebo reference="front_axle_link">
-    <material>Gazebo/FlatBlack</material>
-    <turnGravityOff>false</turnGravityOff>
-  </gazebo>
-  <!-- Front wheels -->
-  <grizzly_wheel fb="front"
-                 lr="left"
-                 parent="front_axle_link"
-                 translateX="0"
-                 translateY="1.75"
-                 translateZ="0"
-                 flipY="0" />
-  <grizzly_wheel fb="front"
-                 lr="right"
-                 parent="front_axle_link"
-                 translateX="0"
-                 translateY="-1.75"
-                 translateZ="0"
-                 flipY="1" />
-  <!-- Grizzly Plugin -->
-  <gazebo>
-    <plugin name="grizzly_diff_controller"
-            filename="libgrizzly_gazebo_plugins.so">
-      <alwaysOn>true</alwaysOn>
-      <updateRate>100.0</updateRate>
-      <backLeftJoint>joint_back_left_wheel</backLeftJoint>
-      <backRightJoint>joint_back_right_wheel</backRightJoint>
-      <frontLeftJoint>joint_front_left_wheel</frontLeftJoint>
-      <frontRightJoint>joint_front_right_wheel</frontRightJoint>
-      <frontAxleJoint>front_axle_joint</frontAxleJoint>
-      <wheelSeparation>${base_y_size}</wheelSeparation>
-      <wheelDiameter>${wheel_x_size}</wheelDiameter>
-      <torque>35</torque>
-    </plugin>
-  </gazebo>
+  <grizzly_wheel fr="front" lr="left" parent="front_axle_link"
+                 translateX="0" translateY="1" flipY="0" />
+  <grizzly_wheel fr="front" lr="right" parent="front_axle_link"
+                 translateX="0" translateY="-1" flipY="1" />
+  <grizzly_wheel fr="rear" lr="left" parent="chassis_link"
+                 translateX="-1" translateY="1" flipY="0" />
+  <grizzly_wheel fr="rear" lr="right" parent="chassis_link"
+                 translateX="-1" translateY="-1" flipY="1" />
 </robot>

File: grizzly_description/urdf/materials.urdf.xacro (robot description, xacro)
@@ -35,9 +35,9 @@
     <color rgba="0.0 0.8 0.0 1.0" />
   </material>
-  <material name="Gray">
-    <color rgba="0.7 0.7 0.7 1.0" />
+  <material name="Grey">
+    <color rgba="0.3 0.3 0.3 1.0" />
   </material>
-  <material name="DarkGray">
-    <color rgba="0.3 0.3 0.3 1.0" />
+  <material name="DarkGrey">
+    <color rgba="0.2 0.2 0.2 1.0" />
   </material>
   <material name="Red">

File: grizzly_description/urdf/wheel.urdf.xacro (robot description, xacro)
@@ -2,4 +2,5 @@
 <!--
 Copyright (c) 2012, Siddhant Ahuja (Sid)
+Copyright (c) 2014, Clearpath Robotics
 All rights reserved.
 Redistribution and use in source and binary forms, with or without
@@ -25,70 +26,17 @@
 This program contains the description of the robot wheel model for Clearpath Grizzly
 -->
-<robot xmlns:sensor="http://playerstage.sourceforge.net/gazebo/xmlschema/#sensor"
-       xmlns:controller="http://playerstage.sourceforge.net/gazebo/xmlschema/#controller"
-       xmlns:interface="http://playerstage.sourceforge.net/gazebo/xmlschema/#interface"
-       xmlns:xacro="http://ros.org/wiki/xacro"
-       name="grizzly_wheel">
-  <property name="M_PI"
-            value="3.14159" />
-  <!-- Wheel -->
-  <property name="wheel_x_com"
-            value="0.00000000" />
-  <!-- com : center of mass -->
-  <property name="wheel_y_com"
-            value="0.00000000" />
-  <!-- com : center of mass -->
-  <property name="wheel_z_com"
-            value="0.00019000" />
-  <!-- com : center of mass -->
-  <property name="wheel_x_size"
-            value="0.66" />
-  <property name="wheel_y_size"
-            value="0.66" />
-  <property name="wheel_z_size"
-            value="0.252" />
-  <property name="wheel_mass"
-            value="2.63657000" />
-  <!-- in kg-->
-  <property name="wheel_ixx_com_cs"
-            value="0.02466885" />
-  <!-- at center of mass aligned with coordinate system, kg*m^2-->
-  <property name="wheel_ixy_com_cs"
-            value="0.00000000" />
-  <!-- at center of mass aligned with coordinate system, kg*m^2-->
-  <property name="wheel_ixz_com_cs"
-            value="0.00000000" />
-  <!-- at center of mass aligned with coordinate system, kg*m^2-->
-  <property name="wheel_iyy_com_cs"
-            value="0.02466885" />
-  <!-- at center of mass aligned with coordinate system, kg*m^2-->
-  <property name="wheel_iyz_com_cs"
-            value="0.00000000" />
-  <!-- at center of mass aligned with coordinate system, kg*m^2-->
-  <property name="wheel_izz_com_cs"
-            value="0.04410576" />
-  <!-- at center of mass aligned with coordinate system, kg*m^2-->
-  <property name="base_x_origin_to_wheel_origin"
-            value="0.25600006" />
-  <property name="base_y_origin_to_wheel_origin"
-            value="0.285475" />
-  <property name="base_z_origin_to_wheel_origin"
-            value="0.0" />
-  <property name="base_z_origin_offset"
-            value="0.2" />
-  <!-- origin is offset in + z direction by 3.175mm, so need to bring it back down for visual and collision-->
+<robot name="grizzly_wheel" xmlns:xacro="http://ros.org/wiki/xacro">
+  <property name="wheel_mass" value="15" />
+  <property name="wheel_radius" value="0.33" />
+  <property name="wheel_width" value="0.252" />
   <xacro:macro name="grizzly_wheel"
-               params="fb lr parent translateX translateY translateZ flipY">
-    <!--fb : front, back ; lr: left, right -->
-    <link name="${fb}_${lr}_wheel">
+               params="fr lr parent translateX translateY flipY">
+    <!--fr : front, rear ; lr: left, right -->
+    <link name="${fr}_${lr}_wheel">
       <inertial>
         <mass value="${wheel_mass}" />
-        <origin xyz="${wheel_x_com} ${wheel_y_com} ${wheel_z_com}" />
-        <inertia ixx="${wheel_ixx_com_cs}"
-                 ixy="${wheel_ixy_com_cs}"
-                 ixz="${wheel_ixz_com_cs}"
-                 iyy="${wheel_iyy_com_cs}"
-                 iyz="${wheel_iyz_com_cs}"
-                 izz="${wheel_izz_com_cs}" />
+        <origin xyz="-0.002 -0.198 0.003" />
+        <inertia ixx="14.68" ixy="-0.033" ixz="0.07"
+                 iyy="26.7" iyz="-0.05" izz="14.68" />
       </inertial>
       <visual>
@@ -98,5 +46,5 @@
           <mesh filename="package://grizzly_description/meshes/wheel.stl" />
         </geometry>
-        <material name="DarkGray" />
+        <material name="Grey" />
       </visual>
       <collision>
@@ -104,12 +52,12 @@
                 rpy="${M_PI/2} ${flipY*M_PI} 0" />
         <geometry>
-          <cylinder length="${wheel_z_size}"
-                    radius="${wheel_x_size/2}" />
+          <cylinder length="${wheel_width}"
+                    radius="${wheel_radius}" />
         </geometry>
       </collision>
     </link>
-    <gazebo reference="${fb}_${lr}_wheel">
-      <mu1 value="100.0" />
-      <mu2 value="0.1" />
+    <gazebo reference="${fr}_${lr}_wheel">
+      <mu1 value="1.0" />
+      <mu2 value="1.0" />
       <kp value="10000000.0" />
       <kd value="1.0" />
@@ -117,10 +65,11 @@
       <material>Gazebo/Grey</material>
       <turnGravityOff>false</turnGravityOff>
+      <selfCollide>true</selfCollide>
     </gazebo>
-    <joint name="joint_${fb}_${lr}_wheel"
+    <joint name="joint_${fr}_${lr}_wheel"
            type="continuous">
       <parent link="${parent}" />
-      <child link="${fb}_${lr}_wheel" />
-      <origin xyz="${translateX * base_x_origin_to_wheel_origin} ${translateY * base_y_origin_to_wheel_origin} ${translateZ}"
+      <child link="${fr}_${lr}_wheel" />
+      <origin xyz="${translateX * base_x_origin_to_wheel_origin} ${translateY * base_y_origin_to_wheel_origin} 0"
               rpy="0 0 0" />
       <axis xyz="0 1 0"
@@ -131,12 +80,13 @@
                         friction="0.0" />
     </joint>
-    <!-- Transmission is important to link the joints and the controller -->
-    <transmission name="joint_${fb}_${lr}_wheel_trans"
+    <!-- Transmission links the joints and the controller -->
+<!--     <transmission name="joint_${fr}_${lr}_wheel_trans"
                   type="SimpleTransmission">
-      <actuator name="joint_${fb}_${lr}_wheel_motor" />
-      <joint name="joint_${fb}_${lr}_wheel" />
-      <mechanicalReduction>1</mechanicalReduction>
-      <motorTorqueConstant>1</motorTorqueConstant>
-    </transmission>
+      <actuator name="joint_${fr}_${lr}_wheel_motor" >
+          <mechanicalReduction>1</mechanicalReduction>
+          <motorTorqueConstant>1</motorTorqueConstant>
+      </actuator>
+      <joint name="joint_${fr}_${lr}_wheel" />
+    </transmission> -->
   </xacro:macro>
 </robot>
