Commit message: Imported upstream version '0.4.1' of 'upstream'

File: grizzly_description/urdf/accessories.urdf.xacro (robot description, xacro)
@@ -1,19 +1,75 @@
 <?xml version="1.0"?>
 <robot name="grizzly_accessories" xmlns:xacro="http://ros.org/wiki/xacro">
+  <xacro:include filename="$(find velodyne_description)/urdf/HDL-32E.urdf.xacro"/>
+  <xacro:include filename="$(find flir_ptu_description)/urdf/d46.urdf.xacro" />
+  <xacro:include filename="$(find pointgrey_camera_description)/urdf/pointgrey_bumblebee2.urdf.xacro" />
+  <xacro:include filename="$(find lms1xx)/urdf/sick_lms1xx.urdf.xacro" />
+  <xacro:arg name="ptu_enabled" default="$(optenv GRIZZLY_PTU_ENABLED false)" />
+  <xacro:arg name="ptu_parent_link" default="$(optenv GRIZZLY_PTU_PARENT_LINK front_sensor_mount_link)" />
+  <xacro:arg name="ptu_xyz" default="$(optenv GRIZZLY_PTU_XYZ 0.0 0.0 0.0)" />
+  <xacro:arg name="ptu_rpy" default="$(optenv GRIZZLY_PTU_RPY 3.14159 0 0)" />
+  <xacro:arg name="hdl32_enabled" default="$(optenv GRIZZLY_HDL32_ENABLED false)" />
+  <xacro:arg name="hdl32_parent_link" default="$(optenv GRIZZLY_HDL32_PARENT_LINK front_sensor_mount_link)" />
+  <xacro:arg name="hdl32_xyz" default="$(optenv GRIZZLY_HDL32_XYZ 0 0 0.003175)" />
+  <xacro:arg name="hdl32_rpy" default="$(optenv GRIZZLY_HDL32_RPY 0.0 0.0 -1.5708)" />
+  <xacro:arg name="bb2_enabled" default="$(optenv GRIZZLY_BB2_ENABLED false)" />
+  <xacro:arg name="bb2_parent_link" default="$(optenv GRIZZLY_BB2_PARENT_LINK ptu_mount_link)" />
+  <xacro:arg name="bb2_xyz" default="$(optenv GRIZZLY_BB2_XYZ 0.0 0.0 0.0)" />
+  <xacro:arg name="bb2_rpy" default="$(optenv GRIZZLY_BB2_RPY 0.0 0.0 0.0)" />
+  <xacro:arg name="lms_enabled" default="$(optenv GRIZZLY_LMS_ENABLED false)" />
+  <xacro:arg name="lms_parent_link" default="$(optenv GRIZZLY_LMS_PARENT_LINK sensor_anchor_link)" />
+  <xacro:arg name="lms_xyz" default="$(optenv GRIZZLY_LMS_XYZ 0.78 0.0 0.08)" />
+  <xacro:arg name="lms_rpy" default="$(optenv GRIZZLY_LMS_RPY 0.0 0.0 0.0)" />
+  <xacro:arg name="lms_mount_angle" default="$(optenv GRIZZLY_LMS_ANGLE 0.523599)" />
   <xacro:macro name="grizzly_decorate">
-<!-- Purely decorative visual component. -->
-  <link name="fenders_link">
-    <visual>
-      <origin xyz="0 0 ${ground_clearance}" rpy="${M_PI/2} 0 ${M_PI/2}"/>
-      <geometry>
-        <mesh filename="package://grizzly_description/meshes/bumper.stl" />
-      </geometry>
-      <material name="Yellow" />
-    </visual>
-  </link>
-  <joint name="fenders_joint" type="fixed">
-    <parent link="chassis_link" />
-    <child link="fenders_link" />
-  </joint>
+    <!-- Purely decorative visual component. -->
+    <link name="fenders_link">
+      <visual>
+        <origin xyz="0 0 ${ground_clearance}" rpy="${M_PI/2} 0 ${M_PI/2}"/>
+        <geometry>
+          <mesh filename="package://grizzly_description/meshes/bumper.stl" />
+        </geometry>
+        <material name="Yellow" />
+      </visual>
+    </link>
+    <joint name="fenders_joint" type="fixed">
+      <parent link="chassis_link" />
+      <child link="fenders_link" />
+    </joint>
+    <xacro:if value="$(arg hdl32_enabled)">
+      <HDL-32E parent="$(arg hdl32_parent_link)" hz="10" samples="220">
+        <origin xyz="$(arg hdl32_xyz)" rpy="$(arg hdl32_rpy)" />
+      </HDL-32E>
+    </xacro:if>
+    <xacro:if value="$(arg ptu_enabled)">
+      <joint name="ptu_mount_joint" type="fixed">
+        <parent link="$(arg ptu_parent_link)"/>
+        <child link="ptu_base_link"/>
+        <origin xyz="$(arg ptu_xyz)" rpy="$(arg ptu_rpy)" />
+      </joint>
+      <ptu_d46 name="ptu"/>
+    </xacro:if>
+    <xacro:if value="$(arg bb2_enabled)">
+      <joint name="bumblebee2_joint" type="fixed">
+        <origin xyz="$(arg bb2_xyz)" rpy="$(arg bb2_rpy)" />
+        <parent link="$(arg bb2_parent_link)" />
+        <child link="bumblebee2" />
+      </joint>
+      <BB2-08S2C-38 frame="bumblebee2" name="bumblebee2" />
+    </xacro:if>
+    <xacro:if value="$(arg lms_enabled)">
+      <joint name="lms_mount_joint" type="fixed">
+        <origin xyz="$(arg lms_xyz)" rpy="$(arg lms_rpy)" />
+        <parent link="$(arg lms_parent_link)" />
+        <child link="lms_mount_link" />
+      </joint>
+      <link name="lms_mount_link" />
+      <joint name="lms_joint" type="fixed">
+        <origin xyz="-0.005 0 -0.0367" rpy="3.14159 $(arg lms_mount_angle) 0.0" />
+        <parent link="lms_mount_link" />
+        <child link="laser" />
+      </joint>
+      <sick_lms1xx/>
+    </xacro:if>
   </xacro:macro>
   <material name="Black">

File: grizzly_description/urdf/grizzly.urdf.xacro (robot description, xacro)
@@ -26,4 +26,11 @@
   <!-- Root link of Grizzly -->
   <link name="base_link" />
+  <!-- Sensor Arch Options -->
+  <xacro:arg name="front_sensor_arch_enabled" default="$(optenv GRIZZLY_FRONT_SENSOR_ARCH_ENABLED false)" />
+  <xacro:arg name="front_tower_xyz" default="$(optenv GRIZZLY_FRONT_SENSOR_ARCH_XYZ 0.495 0.0 0.0)" />
+  <xacro:arg name="front_tower_rpy" default="$(optenv GRIZZLY_FRONT_SENSOR_ARCH_RPY 0.0 0.0 0.0)" />
+  <xacro:arg name="rear_sensor_arch_enabled" default="$(optenv GRIZZLY_REAR_SENSOR_ARCH_ENABLED true)" />
+  <xacro:arg name="rear_tower_xyz" default="$(optenv GRIZZLY_REAR_SENSOR_ARCH_XYZ -0.63 0.0 0.0)" />
+  <xacro:arg name="rear_tower_rpy" default="$(optenv GRIZZLY_REAR_SENSOR_ARCH_RPY 0.0 0.0 0.0)" />
   <!-- Base link is the center of the robot's bottom plate -->
   <link name="chassis_link">
@@ -98,12 +105,4 @@
     <child link="sensor_anchor_link" />
   </joint>
-  <!-- This is the approximate position of the GPS antenna on the standard configuration. -->
-  <link name="navsat_link" />
-  <joint name="navsat_joint" type="fixed">
-    <origin xyz="-${base_x_size/2} 0 0"
-            rpy="0 0 0" />
-    <parent link="sensor_anchor_link" />
-    <child link="navsat_link" />
-  </joint>
   <!-- The position and orientation of the IMU in the rear compartment. -->
   <link name="imu_link" />
@@ -114,41 +113,42 @@
     <child link="imu_link" />
   </joint>
-	<xacro:macro name="grizzly_wheel" params="wheel_prefix parent *joint_pose flipY">
-		<link name="${wheel_prefix}_wheel_link">
-			<inertial>
-			  <mass value="${wheel_mass}" />
-			  <origin xyz="-0.002 -0.198 0.003" />
-			  <inertia  ixx="14.68" ixy="-0.033" ixz="0.07" iyy="26.7" iyz="-0.05" izz="14.68" />
-			</inertial>
-			<visual>
-			  <origin xyz="0 0 0" rpy="${M_PI/2} ${flipY*M_PI} ${M_PI/2}" />
-			  <geometry>
-			    <mesh filename="package://grizzly_description/meshes/wheel.stl" />
-			  </geometry>
-			</visual>
-			<collision>
-			  <origin xyz="0 0 0" rpy="${M_PI/2} ${flipY*M_PI} 0" />
-			  <geometry>
-		  	    <cylinder length="${wheel_width}" radius="${wheel_radius}" />
-			  </geometry>
-			</collision>
-		</link>
-		<joint name="${wheel_prefix}_wheel" type="continuous">
-			<parent link="${parent}"/>
-			<child link="${wheel_prefix}_wheel_link"/>
-			<xacro:insert_block name="joint_pose"/>
-			<axis xyz="0 1 0" rpy="0 0 0" />
-			<joint_properties damping="0.0" friction="0.0" />
-		</joint>
-		<transmission name="${wheel_prefix}_wheel_trans" type="SimpleTransmission">
-			<type>transmission_interface/SimpleTransmission</type>
-			<actuator name="${wheel_prefix}_wheel_motor">
-				<mechanicalReduction>1</mechanicalReduction>
-			</actuator>
-			<joint name="${wheel_prefix}_wheel">
-				<hardwareInterface>hardware_interface/VelocityJointInterface</hardwareInterface>
-			</joint>
-		</transmission>
-	</xacro:macro>
+  <xacro:macro name="grizzly_wheel" params="wheel_prefix parent *joint_pose flipY">
+    <link name="${wheel_prefix}_wheel_link">
+      <inertial>
+        <mass value="${wheel_mass}" />
+        <origin xyz="-0.002 -0.198 0.003" />
+        <inertia  ixx="14.68" ixy="-0.033" ixz="0.07" iyy="26.7" iyz="-0.05" izz="14.68" />
+      </inertial>
+      <visual>
+        <origin xyz="0 0 0" rpy="${M_PI/2} ${flipY*M_PI} ${M_PI/2}" />
+        <geometry>
+          <mesh filename="package://grizzly_description/meshes/wheel.stl" />
+        </geometry>
+        <material name="DarkGrey" />
+      </visual>
+      <collision>
+        <origin xyz="0 0 0" rpy="${M_PI/2} ${flipY*M_PI} 0" />
+        <geometry>
+          <cylinder length="${wheel_width}" radius="${wheel_radius}" />
+        </geometry>
+      </collision>
+    </link>
+    <joint name="${wheel_prefix}_wheel" type="continuous">
+      <parent link="${parent}"/>
+      <child link="${wheel_prefix}_wheel_link"/>
+      <xacro:insert_block name="joint_pose"/>
+      <axis xyz="0 1 0" rpy="0 0 0" />
+      <joint_properties damping="0.0" friction="0.0" />
+    </joint>
+    <transmission name="${wheel_prefix}_wheel_trans" type="SimpleTransmission">
+      <type>transmission_interface/SimpleTransmission</type>
+      <actuator name="${wheel_prefix}_wheel_motor">
+        <mechanicalReduction>1</mechanicalReduction>
+      </actuator>
+      <joint name="${wheel_prefix}_wheel">
+        <hardwareInterface>hardware_interface/VelocityJointInterface</hardwareInterface>
+      </joint>
+    </transmission>
+  </xacro:macro>
   <!-- Grizzly wheel macros -->
   <xacro:grizzly_wheel wheel_prefix="front_left" parent="front_axle_link" flipY="0">
@@ -164,4 +164,126 @@
     <origin xyz="${-wheelbase/2} ${-track} ${wheel_vertical_offset}" rpy="0 0 0" />
   </xacro:grizzly_wheel>
+  <!-- Front Sensor Arch -->
+  <xacro:if value="$(arg front_sensor_arch_enabled)">
+    <link name="front_sensor_base_link">
+      <visual>
+        <origin xyz="0 0 0" rpy="0 0 0" />
+        <geometry>
+          <mesh filename="package://grizzly_description/meshes/sensor_risers.stl" />
+        </geometry>
+        <material name="DarkGrey" />
+      </visual>
+      <collision>
+        <geometry>
+          <mesh filename="package://grizzly_description/meshes/sensor_risers.stl" />
+        </geometry>
+      </collision>
+    </link>
+    <joint name="front_sensor_base_joint" type="fixed">
+      <origin xyz="$(arg front_tower_xyz)" rpy="$(arg rear_tower_rpy)" />
+      <parent link="sensor_anchor_link" />
+      <child link="front_sensor_base_link" />
+    </joint>
+    <link name="front_sensor_arch_link">
+      <visual>
+        <origin xyz="0 0 0" rpy="0 0 0" />
+        <geometry>
+          <mesh filename="package://grizzly_description/meshes/sensor_arch.stl" />
+        </geometry>
+        <material name="DarkGrey" />
+      </visual>
+      <collision>
+        <geometry>
+          <mesh filename="package://grizzly_description/meshes/sensor_arch.stl" />
+        </geometry>
+      </collision>
+    </link>
+    <joint name="front_sensor_arch_joint" type="fixed">
+      <origin xyz="0 0 0.3" rpy="0 0 0" />
+      <parent link="front_sensor_base_link" />
+      <child link="front_sensor_arch_link" />
+    </joint>
+    <link name="front_sensor_mount_link"/>
+    <joint name="front_sensor_mount_joint" type="fixed">
+      <origin xyz="0 0 0.15" rpy="0 0 0" />
+      <parent link="front_sensor_arch_link" />
+      <child link="front_sensor_mount_link" />
+    </joint>
+  </xacro:if>
+  <link name="navsat_link" />
+  <!-- Rear Sensor Arch -->
+  <xacro:if value="$(arg rear_sensor_arch_enabled)">
+    <link name="rear_sensor_base_link">
+      <visual>
+        <origin xyz="0 0 0" rpy="0 0 0" />
+        <geometry>
+          <mesh filename="package://grizzly_description/meshes/sensor_risers.stl" />
+        </geometry>
+        <material name="DarkGrey" />
+      </visual>
+      <collision>
+        <geometry>
+          <mesh filename="package://grizzly_description/meshes/sensor_risers.stl" />
+        </geometry>
+      </collision>
+    </link>
+    <joint name="rear_sensor_base_joint" type="fixed">
+      <origin xyz="$(arg rear_tower_xyz)" rpy="$(arg rear_tower_rpy)" />
+      <parent link="sensor_anchor_link" />
+      <child link="rear_sensor_base_link" />
+    </joint>
+    <link name="rear_sensor_plate_link">
+      <visual>
+        <origin xyz="0 0 0" rpy="0 0 0" />
+        <geometry>
+          <mesh filename="package://grizzly_description/meshes/sensor_plate.stl" />
+        </geometry>
+        <material name="DarkGrey" />
+      </visual>
+      <collision>
+        <geometry>
+          <mesh filename="package://grizzly_description/meshes/sensor_plate.stl" />
+        </geometry>
+      </collision>
+    </link>
+    <joint name="rear_sensor_plate_joint" type="fixed">
+      <origin xyz="0 0 0.3" rpy="0 0 0" />
+      <parent link="rear_sensor_base_link" />
+      <child link="rear_sensor_plate_link" />
+    </joint>
+    <link name="rear_antenna_link">
+      <visual>
+        <origin xyz="0 0 0" rpy="0 0 0" />
+        <geometry>
+          <mesh filename="package://grizzly_description/meshes/antennas.stl" />
+        </geometry>
+        <material name="Grey" />
+      </visual>
+      <collision>
+        <geometry>
+          <mesh filename="package://grizzly_description/meshes/antennas.stl" />
+        </geometry>
+      </collision>
+    </link>
+    <joint name="rear_antenna_joint" type="fixed">
+      <origin xyz="0 0 0.003175" rpy="0 0 0" />
+      <parent link="rear_sensor_plate_link" />
+      <child link="rear_antenna_link" />
+    </joint>
+    <!-- This is the approximate position of the GPS antenna on the standard configuration. -->
+    <joint name="navsat_joint" type="fixed">
+      <origin xyz="0 0 0.4" rpy="0 0 0" />
+      <parent link="rear_sensor_plate_link" />
+      <child link="navsat_link" />
+    </joint>
+  </xacro:if>
+  <xacro:unless value="$(arg rear_sensor_arch_enabled)">
+    <joint name="navsat_joint" type="fixed">
+      <origin xyz="-${base_x_size/2} 0 0"
+              rpy="0 0 0" />
+      <parent link="sensor_anchor_link" />
+      <child link="navsat_link" />
+    </joint>
+  </xacro:unless>
   <xacro:grizzly_decorate />
   <!-- Bring in simulation data for Gazebo. -->
